File: designs/mega_board/led_interface.sch (KiCad schematic (older format))
At the start: 0 parts

Commit message: Some addings and sheet configuration
Parts:
- added D?: PWR, symbol Device:LED
- added D?: P3_100, symbol Device:LED
- added D?: P4_100, symbol Device:LED
- added D?: P3_1000, symbol Device:LED
- added D?: P4_1000, symbol Device:LED
- added D?: 2G_WLAN, symbol Device:LED
- added D?: USB_LED, symbol Device:LED
- added D?: 5G_WLAN1, symbol Device:LED
- added D?: 5G_WLAN0, symbol Device:LED
- added D?: STATUS, symbol Device:LED
- added R? (x10): 330, symbol Device:R
Connections:
- net 3v3: now also D?.2 (A), D?.2 (A), D?.2 (A), D?.2 (A), D?.2 (A), D?.2 (A), D?.2 (A), D?.2 (A), D?.2 (A)
- net STATUS: now also D?.2 (A)
- net ~2G_WLAN: now also R?.2
- net ~5G_WLAN0: now also R?.2
- net ~5G_WLAN1: now also R?.2
- net ~P3_100: now also R?.2
- net ~P3_1000: now also R?.2
- net ~P4_100: now also R?.2
- net ~P4_1000: now also R?.2
- net ~PWR: now also R?.2
- net ~USB_LED: now also R?.2
- new net: D?.1 (K), R?.1 (x10)
- new net GND: R?.2
