File: designs/mega_board/pcie_daughterboard.sch (KiCad schematic (older format))
At the start: 0 parts

Commit message: Some addings and sheet configuration
Parts:
- added C? (x2): 0.1uF, symbol Device:C
- added C?: 470uF, symbol Device:CP
- added R? (x7): 0R, symbol Device:R
- added R?: 1.5k, symbol Device:R
- added R? (x2): NL, symbol Device:R
- added U?: PCIe_Conn, symbol PCIe_Conn:PCIe_Conn
Connections:
- new net: R?.1, U?.1 (PCIE_1)
- new net: R?.2, U?.20 (PCIE_20)
- new net: R?.2, R?.2, U?.22 (PCIE_22)
- new net: R?.1, U?.23 (PCIE_23)
- new net: R?.1, U?.25 (PCIE_25)
- new net: R?.1, U?.31 (PCIE_31)
- new net: R?.1, U?.33 (PCIE_33)
- new net: R?.2, U?.44 (PCIE_44)
- new net 3V3: C?.1, C?.1, R?.1, U?.2 (PCIE_2), U?.24 (PCIE_24), U?.39 (PCIE_39), U?.41 (PCIE_41), U?.52 (PCIE_52)
- new net 5V: C?.1, U?.49 (PCIE_49), U?.51 (PCIE_51)
- new net CLKREQ#: U?.7 (PCIE_7)
- new net DISABLE: R?.1
- new net GND: C?.2, C?.2, C?.2, U?.15 (PCIE_15), U?.18 (PCIE_18), U?.21 (PCIE_21), U?.26 (PCIE_26), U?.27 (PCIE_27), U?.29 (PCIE_29), U?.34 (PCIE_34), U?.35 (PCIE_35), U?.37 (PCIE_37), U?.4 (PCIE_4), U?.40 (PCIE_40), U?.43 (PCIE_43), U?.50 (PCIE_50), U?.9 (PCIE_9)
- new net LED_WLAN: R?.1
- new net PCIe_CLK_N: R?.1, U?.11 (PCIE_11)
- new net PCIe_CLK_P: R?.2, U?.13 (PCIE_13)
- new net PCIe_RST: R?.1
- new net PCIe_RX_N: R?.2
- new net PCIe_RX_P: R?.2
- new net PCIe_TX_N: R?.2
- new net PCIe_TX_P: R?.2
- new net SIM_CLK: U?.12 (PCIE_12)
- new net SIM_DATA: U?.10 (PCIE_10)
- new net SIM_RST: U?.14 (PCIE_14)
- new net SIM_VCC: U?.8 (PCIE_8)
- new net SIM_VPP: U?.16 (PCIE_16)
- new net USB_N: U?.36 (PCIE_36)
- new net USB_P: U?.38 (PCIE_38)
- new net WAKE#: R?.2
- no-connect marks 0 -> 13
