File: designs/mega_board/ethernet_frontend.sch (KiCad schematic (older format))
At the start: 0 parts

Commit message: Ethernet frontend schematic
Parts:
- added C? (x8): 0.1uF, 10V, symbol Device:C
- added C? (x3): 10nF, 2KV, symbol Device:C
- added D? (x8): BS05C, symbol Device:D_TVS
- added Q?: BSS138-7-F, symbol Device:Q_NMOS_DSG
- added Q?: Si4435DDY-T1, symbol Device:Q_PMOS_DSG
- added R? (x8): 75, symbol Device:R
- added R? (x4): 0, symbol Device:R
- added R?: 68k, symbol Device:R
- added R?: 100k, symbol Device:R
- added R?: 4k7, symbol Device:R
- added R?: 47k, symbol Device:R
- added U? (x8): QT48A03, symbol QT48A03:QT48A03
- added U? (x8): 3R420L, symbol 3R420L:3R420L
Connections:
- net labels added: AM_TRX0_N, AM_TRX0_P, AM_TRX1_N, AM_TRX1_P, AM_TRX2_N, AM_TRX2_P, AM_TRX3_N, AM_TRX3_P, AT_TRX0_N, AT_TRX0_P, AT_TRX1_N, AT_TRX1_P, AT_TRX2_N, AT_TRX2_P, AT_TRX3_N, AT_TRX3_P, BM_TRX0_N, BM_TRX0_P, BM_TRX1_N, BM_TRX1_P, BM_TRX2_N, BM_TRX2_P, BM_TRX3_N, BM_TRX3_P, BT_TRX0_N, BT_TRX0_P, BT_TRX1_N, BT_TRX1_P, BT_TRX2_N, BT_TRX2_P, BT_TRX3_N, BT_TRX3_P, GND, GNDA, MCT1-5, MCT2, MCT3, MCT4, MCT6, MCT7, MCT8, POE_12V, POE_INJECTION, POE_INJECTION_EN, POE_OUT
- wire segments 0 -> 263

Commit message: Change RJ45 for double RJ45 shielded
Connections:
- net labels added: DISCHARGE
- net labels removed: GNDA
- wire segments 263 -> 264
Changed lines of the file:
@@
 Connection ~ 4600 2650
-$Comp
-L power:GNDA #PWR?
-U 1 1 5D47BA2F
-P 4150 3050
-F 0 "#PWR?" H 4150 2800 50  0001 C CNN
-F 1 "GNDA" H 4155 2877 50  0000 C CNN
-F 2 "" H 4150 3050 50  0001 C CNN
-F 3 "" H 4150 3050 50  0001 C CNN
-	1    4150 3050
-	1    0    0    -1
-$EndComp
 $Comp
 L QT48A03:QT48A03 U?
@@
 Connection ~ 4600 4450
 $Comp
-L power:GNDA #PWR?
-U 1 1 5D47CF97
-P 4150 4850
-F 0 "#PWR?" H 4150 4600 50  0001 C CNN
-F 1 "GNDA" H 4155 4677 50  0000 C CNN
-F 2 "" H 4150 4850 50  0001 C CNN
-F 3 "" H 4150 4850 50  0001 C CNN
-	1    4150 4850
-	1    0    0    -1
-$EndComp
-$Comp
 L QT48A03:QT48A03 U?
 U 3 1 5D47E738
@@
 Connection ~ 4600 6150
 $Comp
-L power:GNDA #PWR?
-U 1 1 5D47E775
-P 4150 6550
-F 0 "#PWR?" H 4150 6300 50  0001 C CNN
-F 1 "GNDA" H 4155 6377 50  0000 C CNN
-F 2 "" H 4150 6550 50  0001 C CNN
-F 3 "" H 4150 6550 50  0001 C CNN
-	1    4150 6550
-	1    0    0    -1
-$EndComp
-$Comp
 L QT48A03:QT48A03 U?
 U 4 1 5D47E77B
@@
 Connection ~ 4600 7950
 $Comp
-L power:GNDA #PWR?
-U 1 1 5D47E7B8
-P 4150 8350
-F 0 "#PWR?" H 4150 8100 50  0001 C CNN
-F 1 "GNDA" H 4155 8177 50  0000 C CNN
-F 2 "" H 4150 8350 50  0001 C CNN
-F 3 "" H 4150 8350 50  0001 C CNN
-	1    4150 8350
-	1    0    0    -1
-$EndComp
-$Comp
 L QT48A03:QT48A03 U?
 U 5 1 5D481F80
@@
 Connection ~ 10250 2650
 $Comp
-L power:GNDA #PWR?
-U 1 1 5D481FBD
-P 9800 3050
-F 0 "#PWR?" H 9800 2800 50  0001 C CNN
-F 1 "GNDA" H 9805 2877 50  0000 C CNN
-F 2 "" H 9800 3050 50  0001 C CNN
-F 3 "" H 9800 3050 50  0001 C CNN
-	1    9800 3050
-	1    0    0    -1
-$EndComp
-$Comp
 L QT48A03:QT48A03 U?
 U 6 1 5D481FC3
@@
 Connection ~ 10250 4450
 $Comp
-L power:GNDA #PWR?
-U 1 1 5D482000
-P 9800 4850
-F 0 "#PWR?" H 9800 4600 50  0001 C CNN
-F 1 "GNDA" H 9805 4677 50  0000 C CNN
-F 2 "" H 9800 4850 50  0001 C CNN
-F 3 "" H 9800 4850 50  0001 C CNN
-	1    9800 4850
-	1    0    0    -1
-$EndComp
-$Comp
 L QT48A03:QT48A03 U?
 U 7 1 5D482006
@@
 Connection ~ 10250 6150
 $Comp
-L power:GNDA #PWR?
-U 1 1 5D482043
-P 9800 6550
-F 0 "#PWR?" H 9800 6300 50  0001 C CNN
-F 1 "GNDA" H 9805 6377 50  0000 C CNN
-F 2 "" H 9800 6550 50  0001 C CNN
-F 3 "" H 9800 6550 50  0001 C CNN
-	1    9800 6550
-	1    0    0    -1
-$EndComp
-$Comp
 L QT48A03:QT48A03 U?
 U 8 1 5D482049
@@
 	10250 7950 10750 7950
 Connection ~ 10250 7950
-$Comp
-L power:GNDA #PWR?
-U 1 1 5D482086
-P 9800 8350
-F 0 "#PWR?" H 9800 8100 50  0001 C CNN
-F 1 "GNDA" H 9805 8177 50  0000 C CNN
-F 2 "" H 9800 8350 50  0001 C CNN
-F 3 "" H 9800 8350 50  0001 C CNN
-	1    9800 8350
-	1    0    0    -1
-$EndComp
 Text Label 4000 1950 0    50   ~ 0
 MCT1-5
@@
 Wire Wire Line
 	14200 6450 13600 6450
+Text Label 9800 8350 0    50   ~ 0
+DISCHARGE
+Text Label 4150 8350 0    50   ~ 0
+DISCHARGE
+Text Label 4150 6550 0    50   ~ 0
+DISCHARGE
+Text Label 4150 4850 0    50   ~ 0
+DISCHARGE
+Text Label 4150 3050 0    50   ~ 0
+DISCHARGE
+Text Label 9800 3050 0    50   ~ 0
+DISCHARGE
+Text Label 9800 4850 0    50   ~ 0
+DISCHARGE
+Text Label 9800 6550 0    50   ~ 0
+DISCHARGE
+Text Label 2150 1000 0    50   ~ 0
+DISCHARGE
+Text HLabel 1500 1000 0    50   Input ~ 0
+DISCHARGE
+Wire Wire Line
+	2150 1000 1500 1000
 $EndSCHEMATC
