File: designs/mega_board/ethernet_frontend.sch (KiCad schematic (older format))
At the start: 46 parts, among them P1 3R420L, P2 3R420L, P3 3R420L, P4 3R420L, P5 3R420L, P6 3R420L, P7 3R420L, P8 3R420L, Q11 BSS138-7-F, Q9 Si4435DDY-T1, T1 QT48A03

Commit message: Add BOM definition for components. We need more iformation for all the components that are not defined.
Parts:
- Q11: Manufacturer (none) -> Diodes Incorporated; Manufacturer PN (none) -> BSS138-7-F; Supplier (none) -> DigiKey; Supplier PN (none) -> BSS138-FDIDKR-ND
- Q9: Manufacturer (none) -> Vishay Siliconix; Manufacturer PN (none) -> SI4435DDY-T1-E3; Supplier (none) -> DigiKey; Supplier PN (none) -> SI4435DDY-T1-E3DKR-ND
Changed lines of the file:
@@
 F 2 "LibreRouter_MegaBoard:SI4435" H 13400 6450 50  0001 C CNN
 F 3 "" H 13400 6450 50  0001 C CNN
+F 4 "Vishay Siliconix" H 13400 6450 50  0001 C CNN "Manufacturer"
+F 5 "SI4435DDY-T1-E3" H 13400 6450 50  0001 C CNN "Manufacturer PN"
+F 6 "DigiKey" H 13400 6450 50  0001 C CNN "Supplier"
+F 7 "SI4435DDY-T1-E3DKR-ND" H 13400 6450 50  0001 C CNN "Supplier PN"
 	1    13400 6450
 	0    -1   -1   0
@@
 F 2 "LibreRouter_MegaBoard:SOT-23" H 13300 8100 50  0001 C CNN
 F 3 "" H 13300 8100 50  0001 C CNN
+F 4 "Diodes Incorporated" H 13300 8100 50  0001 C CNN "Manufacturer"
+F 5 "BSS138-7-F" H 13300 8100 50  0001 C CNN "Manufacturer PN"
+F 6 "DigiKey" H 13300 8100 50  0001 C CNN "Supplier"
+F 7 "BSS138-FDIDKR-ND" H 13300 8100 50  0001 C CNN "Supplier PN"
 	1    13300 8100
 	-1   0    0    -1
