File: designs/mega_board/ethernet_frontend.sch (KiCad schematic (older format))
At the start: 46 parts, among them P1 3R420L, P2 3R420L, P3 3R420L, P4 3R420L, P5 3R420L, P6 3R420L, P7 3R420L, P8 3R420L, Q11 BSS138-7-F, Q9 Si4435DDY-T1, T1 QT48A03

Commit message: Add some missing BOM details for components that are not in common suppliers
Parts:
- D10, D11, D3, D4, D6, D7, D8, D9: Manufacturer (none) -> Bincheng Electronics; Manufacturer PN (none) -> BV05C
- P1, P2, P3, P4, P5, P6, P7, P8: Manufacturer (none) -> Bincheng Electronics; Manufacturer PN (none) -> LTB3D090L
- T1: Manufacturer (none) -> TNK
Changed lines of the file:
@@
 F 2 "LibreRouter_MegaBoard:QT48103" H 4050 3400 50  0001 C CNN
 F 3 "" H 4050 3400 50  0001 C CNN
+F 4 "TNK" H 3200 2400 50  0001 C CNN "Manufacturer"
 	1    3200 2400
 	1    0    0    -1
@@
 F 3 "~" H 1700 2400 50  0001 C CNN
 F 4 "DigiKey" H 1700 2400 50  0001 C CNN "Supplier"
+F 5 "Bincheng Electronics" H 1700 2400 50  0001 C CNN "Manufacturer"
+F 6 "BV05C" H 1700 2400 50  0001 C CNN "Manufacturer PN"
 	1    1700 2400
 	0    1    1    0
@@
 F 2 "LibreRouter_MegaBoard:GDT-LT-B3D090L" H 4600 2400 50  0001 C CNN
 F 3 "" H 4600 2400 50  0001 C CNN
+F 4 "Bincheng Electronics" H 4600 2400 50  0001 C CNN "Manufacturer"
+F 5 "LTB3D090L" H 4600 2400 50  0001 C CNN "Manufacturer PN"
 	1    4600 2400
 	1    0    0    -1
@@
 F 2 "LibreRouter_MegaBoard:QT48103" H 4050 5200 50  0001 C CNN
 F 3 "" H 4050 5200 50  0001 C CNN
+F 4 "TNK" H 3200 4200 50  0001 C CNN "Manufacturer"
 	2    3200 4200
 	1    0    0    -1
@@
 F 3 "~" H 1700 4200 50  0001 C CNN
 F 4 "DigiKey" H 1700 4200 50  0001 C CNN "Supplier"
+F 5 "Bincheng Electronics" H 1700 4200 50  0001 C CNN "Manufacturer"
+F 6 "BV05C" H 1700 4200 50  0001 C CNN "Manufacturer PN"
 	1    1700 4200
 	0    1    1    0
@@
 F 2 "LibreRouter_MegaBoard:GDT-LT-B3D090L" H 4600 4200 50  0001 C CNN
 F 3 "" H 4600 4200 50  0001 C CNN
+F 4 "Bincheng Electronics" H 4600 4200 50  0001 C CNN "Manufacturer"
+F 5 "LTB3D090L" H 4600 4200 50  0001 C CNN "Manufacturer PN"
 	1    4600 4200
 	1    0    0    -1
@@
 F 2 "LibreRouter_MegaBoard:QT48103" H 4050 6900 50  0001 C CNN
 F 3 "" H 4050 6900 50  0001 C CNN
+F 4 "TNK" H 3200 5900 50  0001 C CNN "Manufacturer"
 	3    3200 5900
 	1    0    0    -1
@@
 F 3 "~" H 1700 5900 50  0001 C CNN
 F 4 "DigiKey" H 1700 5900 50  0001 C CNN "Supplier"
+F 5 "Bincheng Electronics" H 1700 5900 50  0001 C CNN "Manufacturer"
+F 6 "BV05C" H 1700 5900 50  0001 C CNN "Manufacturer PN"
 	1    1700 5900
 	0    1    1    0
@@
 F 2 "LibreRouter_MegaBoard:GDT-LT-B3D090L" H 4600 5900 50  0001 C CNN
 F 3 "" H 4600 5900 50  0001 C CNN
+F 4 "Bincheng Electronics" H 4600 5900 50  0001 C CNN "Manufacturer"
+F 5 "LTB3D090L" H 4600 5900 50  0001 C CNN "Manufacturer PN"
 	1    4600 5900
 	1    0    0    -1
@@
 F 2 "LibreRouter_MegaBoard:QT48103" H 4050 8700 50  0001 C CNN
 F 3 "" H 4050 8700 50  0001 C CNN
+F 4 "TNK" H 3200 7700 50  0001 C CNN "Manufacturer"
 	4    3200 7700
 	1    0    0    -1
@@
 F 3 "~" H 1700 7700 50  0001 C CNN
 F 4 "DigiKey" H 1700 7700 50  0001 C CNN "Supplier"
+F 5 "Bincheng Electronics" H 1700 7700 50  0001 C CNN "Manufacturer"
+F 6 "BV05C" H 1700 7700 50  0001 C CNN "Manufacturer PN"
 	1    1700 7700
 	0    1    1    0
@@
 F 2 "LibreRouter_MegaBoard:GDT-LT-B3D090L" H 4600 7700 50  0001 C CNN
 F 3 "" H 4600 7700 50  0001 C CNN
+F 4 "Bincheng Electronics" H 4600 7700 50  0001 C CNN "Manufacturer"
+F 5 "LTB3D090L" H 4600 7700 50  0001 C CNN "Manufacturer PN"
 	1    4600 7700
 	1    0    0    -1
@@
 F 2 "LibreRouter_MegaBoard:QT48103" H 9700 3400 50  0001 C CNN
 F 3 "" H 9700 3400 50  0001 C CNN
+F 4 "TNK" H 8850 2400 50  0001 C CNN "Manufacturer"
 	5    8850 2400
 	1    0    0    -1
@@
 F 3 "~" H 7350 2400 50  0001 C CNN
 F 4 "DigiKey" H 7350 2400 50  0001 C CNN "Supplier"
+F 5 "Bincheng Electronics" H 7350 2400 50  0001 C CNN "Manufacturer"
+F 6 "BV05C" H 7350 2400 50  0001 C CNN "Manufacturer PN"
 	1    7350 2400
 	0    1    1    0
@@
 F 2 "LibreRouter_MegaBoard:GDT-LT-B3D090L" H 10250 2400 50  0001 C CNN
 F 3 "" H 10250 2400 50  0001 C CNN
+F 4 "Bincheng Electronics" H 10250 2400 50  0001 C CNN "Manufacturer"
+F 5 "LTB3D090L" H 10250 2400 50  0001 C CNN "Manufacturer PN"
 	1    10250 2400
 	1    0    0    -1
@@
 F 2 "LibreRouter_MegaBoard:QT48103" H 9700 5200 50  0001 C CNN
 F 3 "" H 9700 5200 50  0001 C CNN
+F 4 "TNK" H 8850 4200 50  0001 C CNN "Manufacturer"
 	6    8850 4200
 	1    0    0    -1
@@
 F 3 "~" H 7350 4200 50  0001 C CNN
 F 4 "DigiKey" H 7350 4200 50  0001 C CNN "Supplier"
+F 5 "Bincheng Electronics" H 7350 4200 50  0001 C CNN "Manufacturer"
+F 6 "BV05C" H 7350 4200 50  0001 C CNN "Manufacturer PN"
 	1    7350 4200
 	0    1    1    0
@@
 F 2 "LibreRouter_MegaBoard:GDT-LT-B3D090L" H 10250 4200 50  0001 C CNN
 F 3 "" H 10250 4200 50  0001 C CNN
+F 4 "Bincheng Electronics" H 10250 4200 50  0001 C CNN "Manufacturer"
+F 5 "LTB3D090L" H 10250 4200 50  0001 C CNN "Manufacturer PN"
 	1    10250 4200
 	1    0    0    -1
@@
 F 2 "LibreRouter_MegaBoard:QT48103" H 9700 6900 50  0001 C CNN
 F 3 "" H 9700 6900 50  0001 C CNN
+F 4 "TNK" H 8850 5900 50  0001 C CNN "Manufacturer"
 	7    8850 5900
 	1    0    0    -1
@@
 F 3 "~" H 7350 5900 50  0001 C CNN
 F 4 "DigiKey" H 7350 5900 50  0001 C CNN "Supplier"
+F 5 "Bincheng Electronics" H 7350 5900 50  0001 C CNN "Manufacturer"
+F 6 "BV05C" H 7350 5900 50  0001 C CNN "Manufacturer PN"
 	1    7350 5900
 	0    1    1    0
@@
 F 2 "LibreRouter_MegaBoard:GDT-LT-B3D090L" H 10250 5900 50  0001 C CNN
 F 3 "" H 10250 5900 50  0001 C CNN
+F 4 "Bincheng Electronics" H 10250 5900 50  0001 C CNN "Manufacturer"
+F 5 "LTB3D090L" H 10250 5900 50  0001 C CNN "Manufacturer PN"
 	1    10250 5900
 	1    0    0    -1
@@
 F 2 "LibreRouter_MegaBoard:QT48103" H 9700 8700 50  0001 C CNN
 F 3 "" H 9700 8700 50  0001 C CNN
+F 4 "TNK" H 8850 7700 50  0001 C CNN "Manufacturer"
 	8    8850 7700
 	1    0    0    -1
@@
 F 3 "~" H 7350 7700 50  0001 C CNN
 F 4 "DigiKey" H 7350 7700 50  0001 C CNN "Supplier"
+F 5 "Bincheng Electronics" H 7350 7700 50  0001 C CNN "Manufacturer"
+F 6 "BV05C" H 7350 7700 50  0001 C CNN "Manufacturer PN"
 	1    7350 7700
 	0    1    1    0
@@
 F 2 "LibreRouter_MegaBoard:GDT-LT-B3D090L" H 10250 7700 50  0001 C CNN
 F 3 "" H 10250 7700 50  0001 C CNN
+F 4 "Bincheng Electronics" H 10250 7700 50  0001 C CNN "Manufacturer"
+F 5 "LTB3D090L" H 10250 7700 50  0001 C CNN "Manufacturer PN"
 	1    10250 7700
 	1    0    0    -1

Commit message: Fix schematic to pcb coherence.
    * Net names on pcb reasigned to new names.
    * Footprint pad names reasigned on lib
    * Fill zones net asociation reasigned
Parts:
- D10, D11, D3, D4, D6, D7, D8, D9: footprint LibreRouter_MegaBoard:SOD−323 -> LibreRouter_MegaBoard:SOD-323
Changed lines of the file:
@@
 F 0 "D9" V 1654 2479 50  0000 L CNN
 F 1 "BS05C" V 1745 2479 50  0000 L CNN
-F 2 "LibreRouter_MegaBoard:SOD−323" H 1700 2400 50  0001 C CNN
+F 2 "LibreRouter_MegaBoard:SOD-323" H 1700 2400 50  0001 C CNN
 F 3 "~" H 1700 2400 50  0001 C CNN
 F 4 "DigiKey" H 1700 2400 50  0001 C CNN "Supplier"
@@
 F 0 "D8" V 1654 4279 50  0000 L CNN
 F 1 "BS05C" V 1745 4279 50  0000 L CNN
-F 2 "LibreRouter_MegaBoard:SOD−323" H 1700 4200 50  0001 C CNN
+F 2 "LibreRouter_MegaBoard:SOD-323" H 1700 4200 50  0001 C CNN
 F 3 "~" H 1700 4200 50  0001 C CNN
 F 4 "DigiKey" H 1700 4200 50  0001 C CNN "Supplier"
@@
 F 0 "D10" V 1654 5979 50  0000 L CNN
 F 1 "BS05C" V 1745 5979 50  0000 L CNN
-F 2 "LibreRouter_MegaBoard:SOD−323" H 1700 5900 50  0001 C CNN
+F 2 "LibreRouter_MegaBoard:SOD-323" H 1700 5900 50  0001 C CNN
 F 3 "~" H 1700 5900 50  0001 C CNN
 F 4 "DigiKey" H 1700 5900 50  0001 C CNN "Supplier"
@@
 F 0 "D11" V 1654 7779 50  0000 L CNN
 F 1 "BS05C" V 1745 7779 50  0000 L CNN
-F 2 "LibreRouter_MegaBoard:SOD−323" H 1700 7700 50  0001 C CNN
+F 2 "LibreRouter_MegaBoard:SOD-323" H 1700 7700 50  0001 C CNN
 F 3 "~" H 1700 7700 50  0001 C CNN
 F 4 "DigiKey" H 1700 7700 50  0001 C CNN "Supplier"
@@
 F 0 "D4" V 7304 2479 50  0000 L CNN
 F 1 "BS05C" V 7395 2479 50  0000 L CNN
-F 2 "LibreRouter_MegaBoard:SOD−323" H 7350 2400 50  0001 C CNN
+F 2 "LibreRouter_MegaBoard:SOD-323" H 7350 2400 50  0001 C CNN
 F 3 "~" H 7350 2400 50  0001 C CNN
 F 4 "DigiKey" H 7350 2400 50  0001 C CNN "Supplier"
@@
 F 0 "D3" V 7304 4279 50  0000 L CNN
 F 1 "BS05C" V 7395 4279 50  0000 L CNN
-F 2 "LibreRouter_MegaBoard:SOD−323" H 7350 4200 50  0001 C CNN
+F 2 "LibreRouter_MegaBoard:SOD-323" H 7350 4200 50  0001 C CNN
 F 3 "~" H 7350 4200 50  0001 C CNN
 F 4 "DigiKey" H 7350 4200 50  0001 C CNN "Supplier"
@@
 F 0 "D6" V 7304 5979 50  0000 L CNN
 F 1 "BS05C" V 7395 5979 50  0000 L CNN
-F 2 "LibreRouter_MegaBoard:SOD−323" H 7350 5900 50  0001 C CNN
+F 2 "LibreRouter_MegaBoard:SOD-323" H 7350 5900 50  0001 C CNN
 F 3 "~" H 7350 5900 50  0001 C CNN
 F 4 "DigiKey" H 7350 5900 50  0001 C CNN "Supplier"
@@
 F 0 "D7" V 7304 7779 50  0000 L CNN
 F 1 "BS05C" V 7395 7779 50  0000 L CNN
-F 2 "LibreRouter_MegaBoard:SOD−323" H 7350 7700 50  0001 C CNN
+F 2 "LibreRouter_MegaBoard:SOD-323" H 7350 7700 50  0001 C CNN
 F 3 "~" H 7350 7700 50  0001 C CNN
 F 4 "DigiKey" H 7350 7700 50  0001 C CNN "Supplier"

Commit message: Add poe input output dual circuit
Parts:
- removed R25: 0, LibreRouter_MegaBoard:R1206, symbol Device:R
- added D27, D28: MBRS540T3, LibreRouter_MegaBoard:SMC, symbol Device:D_Schottky
- added Q12: Si4435DDY-T1, LibreRouter_MegaBoard:SI4435, symbol p-mosfet_so8:P-MOSFET_SO8
- added R125: 100k, LibreRouter_MegaBoard:R0402, symbol Device:R
- added R126: 68k, LibreRouter_MegaBoard:R0402, symbol Device:R
- added R127: 0 1/10W, LibreRouter_MegaBoard:R0603, symbol Device:R
Connections:
- net GND: no longer R44.2
- net MCT6: now also R127.1
- net POE_INJECT_CTRL: now reaches Q11.1 (D), R32.1
- net POE_INJECT_CTRL: now also R126.1
- net at Q11.3 (G), R3.1: now also R44.2; no longer R44.1
- net POE_INJECTION: no longer names the net of Q9.P$1 (S), Q9.P$2 (S), Q9.P$3 (S), R57.2
- net POE_INJECTION: now also D28.1 (K)
- net POE_INJECTION_EN renamed POE_INJECT_SOFT_EN
- net POE_OUT renamed POE_A
- new net: Q12.P$4 (G), R125.1, R126.2
- new net: D27.1 (K), Q12.P$1 (S), Q12.P$2 (S), Q12.P$3 (S), R125.2
- new net POE_B: Q12.P$5 (D), Q12.P$6 (D), Q12.P$7 (D), Q12.P$8 (D), R127.2
- new net POE_INJECT_HARD_EN: R44.1
- new net POE_INJECT_V: D27.2 (A), D28.2 (A)
Other:
- note added: "POE input-output control"
- moved on the sheet: C10, C11, C137, C33, C34, C35, C37, C40, C41, C49, C5, D10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
